File: esp-4relay-board.brd (EAGLE design)
At the start: 126.8 x 47 mm, 50 parts, among them T1 ST03-5MM, T2 ST02-5MM, T3 ST03-5MM, T4 ST03-5MM, T5 ST03-5MM, T6 LM1117

Commit message: README
Routing:
- net +3V3: track 83.5 -> 78.6 mm
- net N$4: track 25.3 -> 26.9 mm
- net N$27: track 25.2 -> 26.4 mm
- net N$36: track 26.1 -> 27.3 mm
- net N$18: track 24.9 -> 25.9 mm
- net +5V: track 368.2 -> 367.4 mm
Changed lines of the file:
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@@
 <wire x1="68.25" y1="23.5" x2="68.25" y2="19.56" width="1.778" layer="1"/>
 <wire x1="68.25" y1="19.56" x2="60.23" y2="11.54" width="1.778" layer="1"/>
-<wire x1="60.23" y1="11.54" x2="56.94" y2="11.54" width="1.778" layer="1"/>
-<wire x1="47.12" y1="11.54" x2="47.04" y2="11.54" width="1.778" layer="1"/>
-<wire x1="47.04" y1="11.54" x2="45.24" y2="9.74" width="1.778" layer="1"/>
-<wire x1="45.24" y1="9.74" x2="37.495" y2="9.74" width="1.778" layer="1"/>
-<wire x1="37.495" y1="9.74" x2="37.31" y2="9.555" width="1.778" layer="1"/>
+<wire x1="60.23" y1="11.54" x2="54.93" y2="7.76" width="1.778" layer="1"/>
+<wire x1="51.07" y1="7.36" x2="46.89" y2="8.41" width="1.778" layer="1"/>
+<wire x1="46.89" y1="8.41" x2="45.42" y2="9.59" width="1.778" layer="1"/>
+<wire x1="45.42" y1="9.59" x2="37.675" y2="9.59" width="1.778" layer="1"/>
+<wire x1="37.675" y1="9.59" x2="37.31" y2="9.555" width="1.778" layer="1"/>
 <wire x1="53.69" y1="4.7" x2="51.63" y2="4.7" width="1.778" layer="16"/>
 <wire x1="51.63" y1="4.7" x2="51.57" y2="4.64" width="1.778" layer="16"/>
-<wire x1="45.24" y1="9.74" x2="45.24" y2="9.75" width="1.778" layer="1"/>
-<wire x1="45.24" y1="9.75" x2="46.77" y2="11.28" width="1.778" layer="1"/>
-<wire x1="46.77" y1="11.28" x2="46.86" y2="11.28" width="1.778" layer="1"/>
-<wire x1="46.86" y1="11.28" x2="47.12" y2="11.54" width="1.778" layer="1"/>
-<wire x1="47.12" y1="11.54" x2="56.94" y2="11.54" width="1.778" layer="1"/>
-<wire x1="56.94" y1="11.54" x2="56.98" y2="11.5" width="1.778" layer="1"/>
-<wire x1="56.98" y1="11.5" x2="56.98" y2="5.83" width="1.778" layer="1"/>
-<wire x1="56.98" y1="5.83" x2="56.37" y2="5.22" width="1.778" layer="1"/>
-<wire x1="56.37" y1="5.22" x2="54.21" y2="5.22" width="1.778" layer="1"/>
+<wire x1="45.42" y1="9.59" x2="46.06" y2="8.96" width="1.778" layer="1"/>
+<wire x1="46.06" y1="8.96" x2="46.8" y2="8.23" width="1.778" layer="1"/>
+<wire x1="46.8" y1="8.23" x2="46.83" y2="8.5" width="1.778" layer="1"/>
+<wire x1="46.83" y1="8.5" x2="51.07" y2="7.36" width="1.778" layer="1"/>
+<wire x1="51.07" y1="7.36" x2="54.93" y2="7.76" width="1.778" layer="1"/>
+<wire x1="54.93" y1="7.76" x2="55.37" y2="7.08" width="1.778" layer="1"/>
+<wire x1="55.37" y1="7.08" x2="55.21" y2="6.8" width="1.778" layer="1"/>
+<wire x1="55.21" y1="6.8" x2="54.94" y2="6.05" width="1.778" layer="1"/>
+<wire x1="54.94" y1="6.05" x2="54.21" y2="5.22" width="1.778" layer="1"/>
 <wire x1="54.21" y1="5.22" x2="53.69" y2="4.7" width="1.778" layer="1"/>
 </signal>
@@
 <wire x1="41.8" y1="11.99" x2="37.725" y2="11.99" width="1.016" layer="1"/>
 <wire x1="37.725" y1="11.99" x2="37.31" y2="12.095" width="1.016" layer="1"/>
-<wire x1="53.955" y1="22.12" x2="53.955" y2="14.875" width="1.778" layer="16"/>
-<wire x1="53.955" y1="14.875" x2="51.06" y2="11.98" width="1.778" layer="16"/>
-<wire x1="51.06" y1="11.98" x2="37.425" y2="11.98" width="1.778" layer="16"/>
+<wire x1="53.955" y1="22.12" x2="45.285" y2="15.295" width="1.778" layer="16"/>
+<wire x1="45.285" y1="15.295" x2="42.39" y2="12.4" width="1.778" layer="16"/>
+<wire x1="42.39" y1="12.4" x2="37.425" y2="11.98" width="1.778" layer="16"/>
 <wire x1="37.425" y1="11.98" x2="37.31" y2="12.095" width="1.778" layer="16"/>
 </signal>
@@
 <wire x1="116.56" y1="35.12" x2="116.56" y2="31.76" width="1.016" layer="1"/>
 <via x="116.56" y="31.76" extent="1-16" drill="0.6" shape="square"/>
-<wire x1="116.56" y1="31.76" x2="115.68" y2="32.64" width="1.016" layer="16"/>
-<wire x1="115.68" y1="32.64" x2="108.2" y2="32.64" width="1.016" layer="16"/>
-<wire x1="108.2" y1="32.64" x2="106.395" y2="30.835" width="1.016" layer="16"/>
+<wire x1="116.56" y1="31.76" x2="116.32" y2="33.49" width="1.016" layer="16"/>
+<wire x1="116.32" y1="33.49" x2="108.84" y2="33.49" width="1.016" layer="16"/>
+<wire x1="108.84" y1="33.49" x2="106.395" y2="30.835" width="1.016" layer="16"/>
 <wire x1="106.395" y1="30.835" x2="106.395" y2="28.455" width="1.016" layer="16"/>
 </signal>
@@
 <wire x1="101.04" y1="34.985" x2="101.04" y2="31.87" width="1.016" layer="1"/>
 <via x="101.04" y="31.87" extent="1-16" drill="0.6" shape="square"/>
-<wire x1="101.04" y1="31.87" x2="100.13" y2="32.78" width="1.016" layer="16"/>
-<wire x1="100.13" y1="32.78" x2="93.33" y2="32.78" width="1.016" layer="16"/>
-<wire x1="93.33" y1="32.78" x2="91.18" y2="30.63" width="1.016" layer="16"/>
+<wire x1="101.04" y1="31.87" x2="100.52" y2="33.36" width="1.016" layer="16"/>
+<wire x1="100.52" y1="33.36" x2="93.72" y2="33.36" width="1.016" layer="16"/>
+<wire x1="93.72" y1="33.36" x2="91.18" y2="30.63" width="1.016" layer="16"/>
 <wire x1="91.18" y1="30.63" x2="91.18" y2="28.475" width="1.016" layer="16"/>
 </signal>
@@
 <wire x1="84.64" y1="35.175" x2="84.64" y2="31.58" width="1.016" layer="1"/>
 <via x="84.64" y="31.58" extent="1-16" drill="0.6" shape="square"/>
-<wire x1="84.64" y1="31.58" x2="83.77" y2="32.45" width="1.016" layer="16"/>
-<wire x1="83.77" y1="32.45" x2="77.38" y2="32.45" width="1.016" layer="16"/>
-<wire x1="77.38" y1="32.45" x2="74.525" y2="29.595" width="1.016" layer="16"/>
+<wire x1="84.64" y1="31.58" x2="84.2" y2="33.18" width="1.016" layer="16"/>
+<wire x1="84.2" y1="33.18" x2="77.81" y2="33.18" width="1.016" layer="16"/>
+<wire x1="77.81" y1="33.18" x2="74.525" y2="29.595" width="1.016" layer="16"/>
 <wire x1="74.525" y1="29.595" x2="74.525" y2="28.33" width="1.016" layer="16"/>
 </signal>
@@
 <wire x1="69.16" y1="35.255" x2="69.16" y2="31.54" width="1.016" layer="1"/>
 <via x="69.16" y="31.54" extent="1-16" drill="0.6" shape="square"/>
-<wire x1="69.16" y1="31.54" x2="67.88" y2="32.82" width="1.016" layer="16"/>
-<wire x1="67.88" y1="32.82" x2="61.82" y2="32.82" width="1.016" layer="16"/>
-<wire x1="61.82" y1="32.82" x2="59.305" y2="30.305" width="1.016" layer="16"/>
+<wire x1="69.16" y1="31.54" x2="68.86" y2="33.38" width="1.016" layer="16"/>
+<wire x1="68.86" y1="33.38" x2="62.8" y2="33.38" width="1.016" layer="16"/>
+<wire x1="62.8" y1="33.38" x2="59.305" y2="30.305" width="1.016" layer="16"/>
 <wire x1="59.305" y1="30.305" x2="59.305" y2="28.365" width="1.016" layer="16"/>
 </signal>
