File: esp-4relay-board.sch (EAGLE design)
At the start: 50 parts, among them T1 ST03-5MM, T2 ST02-5MM, T3 ST03-5MM, T4 ST03-5MM, T5 ST03-5MM, T6 LM1117

Commit message: no optocops
Parts:
- removed +5V, GND, RXD, TXD: TPTP15R, testpad:TPTP15R
- removed BTN3, BTN4: (no value), PRT-Switch:BUTTON-2PSWITCH-TURTLE-2P
- removed C3: 10uF, SparkFun-Passives:CAP_POLSMD
- removed C5: 100uF, SparkFun-Passives:CAP_POLSMD
- removed OK1, OK2, OK3, OK4: PC817, optocoupler-2:PC817
- removed R9: (no value), resistor:R-EU_R1206
- removed RGPIO2: 10K, PRT-RCL:RESISTORR0805
- removed T6: LM1117, SparkFun-PowerIC:V_REG_LD1117VXX
- removed U$1, U$2, U$3, U$4: RELAYPTH, SRD-05VDC-SL-C:RELAYPTH
- added C2: 100uF, cap-master:CNP-3216
- added C4: 10uF, cap-master:CNP-3216
- added FLASH, RESET: (no value), PRT-Switch:BUTTON-2PSWITCH-TURTLE-2P
- added GOLD_ORB_SM1: OSHWLOGOLOGO16MM, oshw:OSHWLOGOLOGO16MM
- added LM1117: (no value), pinhead:PINHD-1X3
- added PINS, PROG: (no value), pinhead:PINHD-1X5
- added R25: 10K, PRT-RCL:RESISTORR0805
- added R4: (no value), resistor:R-EU_R1206
- added RELAY1, RELAY2, RELAY3, RELAY4: RELAYPTH, SRD-05VDC-SL-C:RELAYPTH
- added RELAYS: (no value), pinhead:PINHD-1X4
- added VREG: HT7333, holtek2:HT7333
- R1, R3, R5, R7: value (none) -> 15K
- U1: device esp8266modules:ESP12 -> esp8266modules:ESP12SMD
Connections:
- removed net N$25: T3.3, U$2.SWOPEN
- removed net N$26: T3.1, U$2.SWCLOSE
- removed net N$27: D3.A, S8050#3.C, U$3.COIL0
- removed net N$29: OK3.EMIT, R6.2
- removed net N$30: R6.1, S8050#3.B
- removed net N$31: OK3.A, R7.2
- removed net N$32: LED3.A, OK3.C
- removed net N$33: T4.2, U$3.SWCOMMON
- removed net N$34: T4.3, U$3.SWOPEN
- removed net N$35: T4.1, U$3.SWCLOSE
- removed net N$36: D4.A, S8050#4.C, U$4.COIL0
- removed net N$38: OK4.EMIT, R8.2
- removed net N$39: R8.1, S8050#4.B
- removed net N$40: OK4.A, R9.2
- removed net N$41: LED4.A, OK4.C
- removed net N$42: T5.2, U$4.SWCOMMON
- removed net N$43: T5.3, U$4.SWOPEN
- removed net N$44: T5.1, U$4.SWCLOSE
- removed net N$8 (its old number): LED1.A, OK1.C
- new net AC1: HKLP1.AC1, T2.1
- new net AC2: HKLP1.AC2, T2.2
- new net GPIO00: FLASH.P$1, R21.2
- new net GPIO02: R25.1
- new net GPIO04: R5.2, RELAYS.2, U1.GPIO4
- new net GPIO05: R7.2, RELAYS.1, U1.GPIO5
- new net N$11: RELAY2.SWCLOSE, T3.1
- new net N$12: RELAY2.SWOPEN, T3.3
- new net N$13: D3.A, LED3.A, RELAY3.COIL1, S8050#3.C
- new net N$14: R5.1, S8050#3.B
- new net N$15: LED3.C, R6.2
- new net N$19: D4.A, LED4.A, RELAY4.COIL1, S8050#4.C
- new net N$21: LED4.C, R8.2
- new net N$5: RELAY1.SWOPEN, T1.3
- new net N$6: D2.A, LED2.A, RELAY2.COIL1, S8050#2.C
- net +3V3: now also C2.2, LM1117.2, PROG.1, R25.2, VREG.OUT; no longer C5.+, RGPIO2.2, T6.OUT
- net +5V: now also C4.2, LM1117.1, PROG.2, R4.1, R6.1, R8.1, RELAY1.COIL0, RELAY2.COIL0, RELAY3.COIL0, RELAY4.COIL0, VREG.IN; no longer +5V.TP, C3.+, OK1.COL, OK2.COL, OK3.COL, OK4.COL, R5.1, R7.1, R9.1, T6.IN, U$1.COIL1, U$2.COIL1, U$3.COIL1, U$4.COIL1
- net GND: now also C2.1, C4.1, FLASH.P$2, LM1117.3, PROG.5, RESET.P$2, VREG.GND; no longer BTN3.P$2, BTN4.P$2, C3.-, C5.-, GND.TP, T6.GND
- net GPIO0: now also PINS.3; no longer BTN4.P$1, R21.2
- net GPIO12: now also PINS.1; no longer LED3.C
- net GPIO13: now also PINS.2; no longer LED4.C
- net GPIO14: now also R3.2, RELAYS.3; no longer LED2.C
- net GPIO15: now also PINS.4
- net GPIO16: now also R1.2, RELAYS.4; no longer LED1.C
- net GPIO2: now also PINS.5; no longer RGPIO2.1
- net N$1: now also RELAY1.SWCLOSE, T1.1; no longer OK1.EMIT, R1.2
- net N$10: now also RELAY2.SWCOMMON, T3.2; no longer T1.1, U$1.SWCLOSE
- net N$16: now also RELAY3.SWCOMMON, T4.2; no longer HKLP1.AC1, T2.2
- net N$17: now also RELAY3.SWCLOSE, T4.1; no longer HKLP1.AC2, T2.1
- net N$18: now also RELAY3.SWOPEN, T4.3; no longer D2.A, S8050#2.C, U$2.COIL0
- net N$20: now also R7.1, S8050#4.B; no longer OK2.EMIT, R3.2
- net N$22: now also RELAY4.SWCOMMON, T5.2; no longer OK2.A, R5.2
- net N$23: now also RELAY4.SWCLOSE, T5.1; no longer LED2.A, OK2.C
- net N$24: now also RELAY4.SWOPEN, T5.3; no longer T3.2, U$2.SWCOMMON
- net N$3: now also RELAY1.SWCOMMON; no longer U$1.SWCOMMON
- net N$4: now also LED1.A, RELAY1.COIL1; no longer U$1.COIL0
- net N$7: now also LED1.C; no longer OK1.A
- net N$9: now also LED2.C, R4.2; no longer T1.3, U$1.SWOPEN
- net RST: now also RESET.P$1; no longer BTN3.P$1
- net RXD: now also PROG.4; no longer RXD.TP
- net TXD: now also PROG.3; no longer TXD.TP
Other:
- note added: "ESP12F/ESP12E/ESP12S"
- note added: "POWER SUPPLY 220VAC => 5VDC => 3V3VDC"
- note added: "RELAYS"
- note added: "RELAYS HEADER"
- note added: "Vedran Alajbegovic www.nardev.org GitHub: https://github.com/nardev/esp4relay"
- moved on the sheet: C1, D1, D2, D3, D4, HKLP1, LED1, LED2, LED3, LED4, R1, R2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
